Commit message: added tcp link

File: robotiq_2f_85_gripper_visualization/urdf/robotiq_arg2f_85_model_macro.xacro (robot description, xacro)
@@ -165,5 +165,5 @@
       <child link="${prefix}left_outer_knuckle" />
       <axis xyz="1 0 0" />
-      <limit lower="0" upper="0.8" velocity="2.0" effort="1000" />
+      <limit lower="0" upper="0.755" velocity="0.7" effort="1000" />
     </joint>
     <xacro:finger_joints prefix="${prefix}" fingerprefix="left" reflect="1.0"/>
@@ -188,4 +188,11 @@
     <xacro:right_outer_knuckle_joint prefix="${prefix}"/>
     <xacro:robotiq_arg2f_transmission prefix="${prefix}"/>
+    <!-- Tool Center Point: Center of the fingertips when gripper is closed -->
+    <joint name="${prefix}tcp_joint" type="fixed">
+      <origin xyz="0 0 0.14" rpy="0 ${-pi/2} 0" />
+      <parent link="${prefix}robotiq_arg2f_base_link" />
+      <child link="${prefix}tcp" />
+    </joint>
+    <link name="${prefix}tcp" />
   </xacro:macro>
 </robot>
